Commit message: force commit

File: urdf/modelo.urdf (robot description, URDF)
Before this commit: robot micarro, 19 links, 18 joints
Joints:
- joint da_link_joint: axis 0.00000 0.00000 1.00000 -> (none); limit lower=-3.14000 upper=3.14000 effort=0.00000 velocity=0.00000 -> (none); type revolute -> fixed
- joint dg_link_joint: axis 0.00000 0.00000 1.00000 -> (none); limit lower=-3.14000 upper=3.14000 effort=0.00000 velocity=0.00000 -> (none); type revolute -> fixed
- joint ia_link_joint: axis 0.00000 0.00000 1.00000 -> (none); limit lower=-3.14000 upper=3.14000 effort=0.00000 velocity=0.00000 -> (none); type revolute -> fixed
- joint ig_link_joint: axis 0.00000 0.00000 1.00000 -> (none); limit lower=-3.14000 upper=3.14000 effort=0.00000 velocity=0.00000 -> (none); type revolute -> fixed
